File: Electrical Schematics/IGCV/FNR v1.4 + Speed v1.2.sch (EAGLE design)
At the start: 40 parts, among them IC3 DPOT, K17 35701331, K18 35701331, K19 G6C-2117P, K20 DF2-L-DC24V, K21 35701331, Q10 BUZ11, Q11 BUZ11, Q5 BUZ11, SW4 Pedal MS, SW6 Pedal MS

Commit message: Updated schematics
Parts:
- removed S13: E-STOP, custom:SWITCH
- removed S4: KEY, custom:SWITCH
- added SW1: (no value), special:SW-C10
- added SW2: Pedal MS, switch-coto:CT10-XXXX-A2
- SW3: value (none) -> Pedal MS; device special:SW-C10 -> switch-coto:CT10-XXXX-A2
- SW4: value Pedal MS -> E-STOP; device switch-coto:CT10-XXXX-A2 -> custom:SWITCH
- SW6: value Pedal MS -> KEY; device switch-coto:CT10-XXXX-A2 -> custom:SWITCH
- renumbered BAT7 to BAT1, BAT8 to BAT2, BAT9 to BAT3, K17 to K2, K18 to K3, K19 to K4, K20 to K1, K21 to K5, OK3 to OK1, Q10 to Q1, Q11 to Q3, Q5 to Q2, R11 to R2, R12 to R1, R13 to R4, R14 to R3, R9 to R5, S14 to SW5, THROTTLE2 to THROTTLE
Connections:
- net B+1: now also SW6.2; no longer S4.2
- net B-: now also SW1.2, SW1.C, SW2.1, SW2.2; no longer SW3.2, SW3.C, SW4.1, SW4.2
- net FGND1: now also SW1.4; no longer SW3.4
- net N$105: now also SW6.1; no longer S4.1
- net N$106: now also SW4.2; no longer S13.2
- net N$122: now also OK1C.COL
- net N$123: now also SW4.1; no longer S13.1
- net N$129: now also SW3.1; no longer SW6.1
- net RGND1: now also SW1.1; no longer SW3.1
- net VCC: now also SW3.2; no longer SW6.2

Commit message: updated schematics
Connections:
- removed net B+1: D12.C, D13.C, D14.C, JP30.1, JP30.2, K21.3, K22.S, K31.3, K41.2, K43.O, K52.P, SW5.2, SW6.2, U$5.B+
- removed net N$106: BAT1.+, K52.S, R5.1, SW4.2
- removed net N$107: R5.2, SW5.1
- removed net N$123: D16.C, K51.3, SW4.1
- new net B+: BAT1.+, D12.C, D13.C, D14.C, D16.C, JP30.1, JP30.2, K21.3, K22.S, K31.3, K41.2, K43.O, K51.3, K52.P, K52.S, R5.1, R5.2, SW5.1, SW5.2, SW6.2, U$5.B+
- new net N$1: D16.A, K51.5, SW4.2
- new net N$2: K13.P, U$5.THROTTLE2
- new net N$3: SW2.1, SW4.1
- net B-: no longer D16.A, K51.5, SW2.1
- net N$111: no longer K13.P, U$5.THROTTLE2
Other:
- moved on the sheet: SW2, SW4, SW5
